Commit message: adding robot sim interface example

File: ros_control_gazebo_tests/models/rr_manipulator.urdf.xacro (robot description, xacro)
@@ -5,5 +5,5 @@
     <plugin
       name="ros_control"
-      filename="libros_control_gazebo_plugin.so"/>
+      filename="$(find ros_control_gazebo_plugin)/lib/libros_control_gazebo_plugin.so"/>
   </gazebo>
   <link name="link1">
@@ -14,5 +14,5 @@
     <visual name="visual">
       <geometry> <box size="10 1 1"/> </geometry>
-      <material> <color rgba="1 0 0 1"/> </material>
+      <material name="red"> <color rgba="1 0 0 1"/> </material>
     </visual>
   </link>
@@ -24,5 +24,5 @@
     <visual name="visual">
       <geometry> <box size="10 1 1"/> </geometry>
-      <material> <color rgba="0.5 0 0.5 1"/> </material>
+      <material name="purple"> <color rgba="1.0 0 1.0 1"/> </material>
     </visual>
   </link>
@@ -34,20 +34,18 @@
     <visual name="visual">
       <geometry> <box size="10 1 1"/> </geometry>
-      <material> <color rgba="0 0 1 1"/> </material>
+      <material name="blue"> <color rgba="0 0 1 1"/> </material>
     </visual>
   </link>
-  <joint name="joint1" type="revolute">
+  <joint name="joint1" type="continuous">
     <parent link="link1"/>
     <child link="link2"/>
     <origin xyz="5 0 0" rpy="0 0 0"/>
     <axis xyz="0 0 1"/>
-    <limit lower="-0.4" upper="0.4"/>
   </joint>
-  <joint name="joint2" type="revolute">
+  <joint name="joint2" type="continuous">
     <parent link="link2"/>
     <child link="link3"/>
     <origin xyz="5 0 0" rpy="0 0 0"/>
     <axis xyz="0 0 1"/>
-    <limit lower="-0.4" upper="0.4"/>
   </joint>
 </robot>

Commit message: working example controller manager and robot sim interface

File: ros_control_gazebo_tests/models/rr_manipulator.urdf.xacro (robot description, xacro)
@@ -1,5 +1,7 @@
 <?xml version="1.0"?>
 <!-- Revolute-Revolute Manipulator -->
-<robot name="rr_manipulator">
+<robot name="rr_manipulator"
+  xmlns:xacro="http://www.ros.org/wiki/xacro">
+  <xacro:property name="PI" value="3.1415926535897931"/>
   <gazebo>
     <plugin
@@ -7,38 +9,74 @@
       filename="$(find ros_control_gazebo_plugin)/lib/libros_control_gazebo_plugin.so"/>
   </gazebo>
+  <material name="red"> <color rgba="1 0 0 1"/> </material>
+  <material name="purple"> <color rgba="1.0 0 1.0 1"/> </material>
+  <material name="blue"> <color rgba="0 0 1 1"/> </material>
+  <link name="world"/>
   <link name="link1">
-    <origin xyz="0 0 0" rpy="0 0 0"/>
     <collision name="collision">
-      <geometry> <box size="10 1 1"/> </geometry>
+      <origin xyz="0.5 0 0" rpy="0 0 0"/>
+      <geometry> <box size="1 0.1 0.1"/> </geometry>
     </collision>
     <visual name="visual">
-      <geometry> <box size="10 1 1"/> </geometry>
-      <material name="red"> <color rgba="1 0 0 1"/> </material>
+      <origin xyz="0.5 0 0" rpy="0 0 0"/>
+      <geometry> <box size="1 0.1 0.1"/> </geometry>
+      <material name="red"/>
     </visual>
+    <inertial>
+      <origin xyz="0.5 0 0" rpy="0 0 0"/>
+      <mass value="1"/>
+      <inertia
+        ixx="1.0" ixy="0.0" ixz="0.0"
+        iyy="1.0" iyz="0.0"
+        izz="1.0"/>
+    </inertial>
   </link>
   <link name="link2">
-    <origin xyz="0 0 0" rpy="0 0 0"/>
     <collision name="collision">
-      <geometry> <box size="10 1 1"/> </geometry>
+      <origin xyz="0.5 0 0" rpy="0 0 0"/>
+      <geometry> <box size="1 0.1 0.1"/> </geometry>
     </collision>
     <visual name="visual">
-      <geometry> <box size="10 1 1"/> </geometry>
-      <material name="purple"> <color rgba="1.0 0 1.0 1"/> </material>
+      <origin xyz="0.5 0 0" rpy="0 0 0"/>
+      <geometry> <box size="1 0.1 0.1"/> </geometry>
+      <material name="purple"/>
     </visual>
+    <inertial>
+      <origin xyz="0.5 0 0" rpy="0 0 0"/>
+      <mass value="1"/>
+      <inertia
+        ixx="1.0" ixy="0.0" ixz="0.0"
+        iyy="1.0" iyz="0.0"
+        izz="1.0"/>
+    </inertial>
   </link>
   <link name="link3">
-    <origin xyz="0 0 0" rpy="0 0 0"/>
     <collision name="collision">
-      <geometry> <box size="10 1 1"/> </geometry>
+      <origin xyz="0.5 0 0" rpy="0 0 0"/>
+      <geometry> <box size="1 0.1 0.1"/> </geometry>
     </collision>
     <visual name="visual">
-      <geometry> <box size="10 1 1"/> </geometry>
-      <material name="blue"> <color rgba="0 0 1 1"/> </material>
+      <origin xyz="0.5 0 0" rpy="0 0 0"/>
+      <geometry> <box size="1 0.1 0.1"/> </geometry>
+      <material name="blue"/>
     </visual>
+    <inertial>
+      <origin xyz="0.5 0 0" rpy="0 0 0"/>
+      <mass value="1"/>
+      <inertia
+        ixx="1.0" ixy="0.0" ixz="0.0"
+        iyy="1.0" iyz="0.0"
+        izz="1.0"/>
+    </inertial>
   </link>
+  <joint name="fixed" type="fixed">
+    <parent link="world"/>
+    <child link="link1"/>
+    <origin xyz="0 0 1" rpy="${PI} 0 0"/>
+  </joint>
   <joint name="joint1" type="continuous">
     <parent link="link1"/>
     <child link="link2"/>
-    <origin xyz="5 0 0" rpy="0 0 0"/>
+    <origin xyz="1 0 0" rpy="0 0 0"/>
     <axis xyz="0 0 1"/>
   </joint>
@@ -46,6 +84,6 @@
     <parent link="link2"/>
     <child link="link3"/>
-    <origin xyz="5 0 0" rpy="0 0 0"/>
-    <axis xyz="0 0 1"/>
+    <origin xyz="1 0 0" rpy="0 0 0"/>
+    <axis xyz="0 1 0"/>
   </joint>
 </robot>

Commit message: Updating urdf to not be stupid, adding anothe readme

File: ros_control_gazebo_tests/models/rr_manipulator.urdf.xacro (robot description, xacro)
@@ -9,4 +9,5 @@
       name="ros_control"
       plugin="$(find ros_control_gazebo_plugin)/lib/libros_control_gazebo_plugin.so">
+      <ns>rr/ros_control</ns>
       <robotSimType>ros_control_gazebo_tests/RobotSimRR</robotSimType>
       <controlPeriod>0.001</controlPeriod>
@@ -20,5 +21,5 @@
     <collision name="collision">
       <origin xyz="0.5 0 0" rpy="0 0 0"/>
-      <geometry> <box size="1 0.1 0.1"/> </geometry>
+      <geometry> <box size="0.9 0.1 0.1"/> </geometry>
     </collision>
     <visual name="visual">
@@ -39,5 +40,5 @@
     <collision name="collision">
       <origin xyz="0.5 0 0" rpy="0 0 0"/>
-      <geometry> <box size="1 0.1 0.1"/> </geometry>
+      <geometry> <box size="0.9 0.1 0.1"/> </geometry>
     </collision>
     <visual name="visual">
@@ -58,5 +59,5 @@
     <collision name="collision">
       <origin xyz="0.5 0 0" rpy="0 0 0"/>
-      <geometry> <box size="1 0.1 0.1"/> </geometry>
+      <geometry> <box size="0.9 0.1 0.1"/> </geometry>
     </collision>
     <visual name="visual">

Commit message: Changed URDF to pendulum-type arm, new run script, new rviz launch file, small plugin tweak

File: ros_control_gazebo_tests/models/rr_manipulator.urdf.xacro (robot description, xacro)
@@ -11,21 +11,18 @@
       <controlPeriod>0.001</controlPeriod>
     </plugin>
+    <material name="red">Gazebo/Red</material>
+    <material name="blue">Gazebo/Blue</material>
   </gazebo>
-  <material name="red"> <color rgba="1 0 0 1"/> </material>
-  <material name="purple"> <color rgba="1.0 0 1.0 1"/> </material>
-  <material name="blue"> <color rgba="0 0 1 1"/> </material>
   <link name="world"/>
   <link name="link1">
-    <collision name="collision">
-      <origin xyz="0.5 0 0" rpy="0 0 0"/>
-      <geometry> <box size="0.9 0.1 0.1"/> </geometry>
-    </collision>
-    <visual name="visual">
-      <origin xyz="0.5 0 0" rpy="0 0 0"/>
-      <geometry> <box size="1 0.1 0.1"/> </geometry>
+    <visual>
+      <origin xyz="0 0 0.5" rpy="0 0 0"/>
+      <geometry>
+	<box size="0.1 0.1 1"/>
+      </geometry>
       <material name="red"/>
     </visual>
     <inertial>
-      <origin xyz="0.5 0 0" rpy="0 0 0"/>
+      <origin xyz="0 0 0.5" rpy="0 0 0"/>
       <mass value="1"/>
       <inertia
@@ -36,15 +33,13 @@
   </link>
   <link name="link2">
-    <collision name="collision">
-      <origin xyz="0.5 0 0" rpy="0 0 0"/>
-      <geometry> <box size="0.9 0.1 0.1"/> </geometry>
-    </collision>
-    <visual name="visual">
-      <origin xyz="0.5 0 0" rpy="0 0 0"/>
-      <geometry> <box size="1 0.1 0.1"/> </geometry>
-      <material name="purple"/>
+    <visual>
+      <origin xyz="0 0 0.45" rpy="0 0 0"/>
+      <geometry>
+	<box size="0.1 0.1 1"/>
+      </geometry>
+      <material name="blue"/>
     </visual>
     <inertial>
-      <origin xyz="0.5 0 0" rpy="0 0 0"/>
+      <origin xyz="0 0 1.5" rpy="0 0 0"/>
       <mass value="1"/>
       <inertia
@@ -55,15 +50,13 @@
   </link>
   <link name="link3">
-    <collision name="collision">
-      <origin xyz="0.5 0 0" rpy="0 0 0"/>
-      <geometry> <box size="0.9 0.1 0.1"/> </geometry>
-    </collision>
-    <visual name="visual">
-      <origin xyz="0.5 0 0" rpy="0 0 0"/>
-      <geometry> <box size="1 0.1 0.1"/> </geometry>
+    <visual>
+      <origin xyz="0 0 0.45" rpy="0 0 0"/>
+      <geometry>
+	<box size="0.1 0.1 1"/>
+      </geometry>
       <material name="blue"/>
     </visual>
     <inertial>
-      <origin xyz="0.5 0 0" rpy="0 0 0"/>
+      <origin xyz="0 0 1.5" rpy="0 0 0"/>
       <mass value="1"/>
       <inertia
@@ -76,16 +69,16 @@
     <parent link="world"/>
     <child link="link1"/>
-    <origin xyz="0 0 1" rpy="${PI} 0 0"/>
+    <!--origin xyz="0 0 1" rpy="${PI} 0 0"/-->
   </joint>
   <joint name="joint1" type="continuous">
     <parent link="link1"/>
     <child link="link2"/>
-    <origin xyz="1 0 0" rpy="0 0 0"/>
-    <axis xyz="0 0 1"/>
+    <origin xyz="0 0.1 0.9" rpy="0 0 0"/>
+    <axis xyz="0 1 0"/>
   </joint>
   <joint name="joint2" type="continuous">
     <parent link="link2"/>
     <child link="link3"/>
-    <origin xyz="1 0 0" rpy="0 0 0"/>
+    <origin xyz="0 0.1 0.9" rpy="0 0 0"/>
     <axis xyz="0 1 0"/>
   </joint>

Commit message: Cleaned up code - no functional changes

File: ros_control_gazebo_tests/models/rr_manipulator.urdf.xacro (robot description, xacro)
@@ -16,4 +16,11 @@
   <link name="world"/>
   <link name="link1">
+    <collision>
+      <origin xyz="0 0 0.5" rpy="0 0 0"/>
+      <geometry>
+	<box size="0.1 0.1 1"/>
+      </geometry>
+      <material name="red"/>
+    </collision>
     <visual>
       <origin xyz="0 0 0.5" rpy="0 0 0"/>
@@ -33,4 +40,11 @@
   </link>
   <link name="link2">
+    <collision>
+      <origin xyz="0 0 0.45" rpy="0 0 0"/>
+      <geometry>
+	<box size="0.1 0.1 1"/>
+      </geometry>
+      <material name="blue"/>
+    </collision>
     <visual>
       <origin xyz="0 0 0.45" rpy="0 0 0"/>
@@ -50,4 +64,11 @@
   </link>
   <link name="link3">
+    <collision>
+      <origin xyz="0 0 0.45" rpy="0 0 0"/>
+      <geometry>
+	<box size="0.1 0.1 1"/>
+      </geometry>
+      <material name="blue"/>
+    </collision>
     <visual>
       <origin xyz="0 0 0.45" rpy="0 0 0"/>
@@ -66,4 +87,8 @@
     </inertial>
   </link>
+  <gazebo reference="link3">
+    <mu1>0.2</mu1>
+    <mu2>0.2</mu2>
+  </gazebo>
   <joint name="fixed" type="fixed">
     <parent link="world"/>

Commit message: fixing errors in doc, making script clearer

File: ros_control_gazebo_tests/models/rr_manipulator.urdf.xacro (robot description, xacro)
@@ -5,4 +5,5 @@
   xmlns:controller="http://playerstage.sourceforge.net/gazebo/xmlschema/#controller">
   <xacro:property name="PI" value="3.1415926535897931"/>
+  <!-- ros_control_gazebo plugin -->
   <gazebo>
     <plugin name="ros_control" filename="libros_control_gazebo_plugin.so">
@@ -19,5 +20,5 @@
       <origin xyz="0 0 0.5" rpy="0 0 0"/>
       <geometry>
-	<box size="0.1 0.1 1"/>
+        <box size="0.1 0.1 1"/>
       </geometry>
       <material name="red"/>
@@ -26,5 +27,5 @@
       <origin xyz="0 0 0.5" rpy="0 0 0"/>
       <geometry>
-	<box size="0.1 0.1 1"/>
+        <box size="0.1 0.1 1"/>
       </geometry>
       <material name="red"/>
@@ -43,5 +44,5 @@
       <origin xyz="0 0 0.45" rpy="0 0 0"/>
       <geometry>
-	<box size="0.1 0.1 1"/>
+        <box size="0.1 0.1 1"/>
       </geometry>
       <material name="blue"/>
@@ -50,5 +51,5 @@
       <origin xyz="0 0 0.45" rpy="0 0 0"/>
       <geometry>
-	<box size="0.1 0.1 1"/>
+        <box size="0.1 0.1 1"/>
       </geometry>
       <material name="blue"/>
@@ -67,5 +68,5 @@
       <origin xyz="0 0 0.45" rpy="0 0 0"/>
       <geometry>
-	<box size="0.1 0.1 1"/>
+        <box size="0.1 0.1 1"/>
       </geometry>
       <material name="blue"/>
@@ -74,5 +75,5 @@
       <origin xyz="0 0 0.45" rpy="0 0 0"/>
       <geometry>
-	<box size="0.1 0.1 1"/>
+        <box size="0.1 0.1 1"/>
       </geometry>
       <material name="blue"/>

Commit message: reverting arm to arm with 3d coupled dynamics

File: ros_control_gazebo_tests/models/rr_manipulator.urdf.xacro (robot description, xacro)
@@ -5,5 +5,4 @@
   xmlns:controller="http://playerstage.sourceforge.net/gazebo/xmlschema/#controller">
   <xacro:property name="PI" value="3.1415926535897931"/>
-  <!-- ros_control_gazebo plugin -->
   <gazebo>
     <plugin name="ros_control" filename="libros_control_gazebo_plugin.so">
@@ -12,25 +11,21 @@
       <controlPeriod>0.001</controlPeriod>
     </plugin>
-    <material name="red">Gazebo/Red</material>
-    <material name="blue">Gazebo/Blue</material>
   </gazebo>
+  <material name="red"> <color rgba="1 0 0 1"/> </material>
+  <material name="purple"> <color rgba="1.0 0 1.0 1"/> </material>
+  <material name="blue"> <color rgba="0 0 1 1"/> </material>
   <link name="world"/>
   <link name="link1">
-    <collision>
-      <origin xyz="0 0 0.5" rpy="0 0 0"/>
-      <geometry>
-        <box size="0.1 0.1 1"/>
-      </geometry>
-      <material name="red"/>
+    <collision name="collision">
+      <origin xyz="0.5 0 0" rpy="0 0 0"/>
+      <geometry> <box size="0.9 0.1 0.1"/> </geometry>
     </collision>
-    <visual>
-      <origin xyz="0 0 0.5" rpy="0 0 0"/>
-      <geometry>
-        <box size="0.1 0.1 1"/>
-      </geometry>
+    <visual name="visual">
+      <origin xyz="0.5 0 0" rpy="0 0 0"/>
+      <geometry> <box size="1 0.1 0.1"/> </geometry>
       <material name="red"/>
     </visual>
     <inertial>
-      <origin xyz="0 0 0.5" rpy="0 0 0"/>
+      <origin xyz="0.5 0 0" rpy="0 0 0"/>
       <mass value="1"/>
       <inertia
@@ -41,20 +36,15 @@
   </link>
   <link name="link2">
-    <collision>
-      <origin xyz="0 0 0.45" rpy="0 0 0"/>
-      <geometry>
-        <box size="0.1 0.1 1"/>
-      </geometry>
-      <material name="blue"/>
+    <collision name="collision">
+      <origin xyz="0.5 0 0" rpy="0 0 0"/>
+      <geometry> <box size="0.9 0.1 0.1"/> </geometry>
     </collision>
-    <visual>
-      <origin xyz="0 0 0.45" rpy="0 0 0"/>
-      <geometry>
-        <box size="0.1 0.1 1"/>
-      </geometry>
-      <material name="blue"/>
+    <visual name="visual">
+      <origin xyz="0.5 0 0" rpy="0 0 0"/>
+      <geometry> <box size="1 0.1 0.1"/> </geometry>
+      <material name="purple"/>
     </visual>
     <inertial>
-      <origin xyz="0 0 1.5" rpy="0 0 0"/>
+      <origin xyz="0.5 0 0" rpy="0 0 0"/>
       <mass value="1"/>
       <inertia
@@ -65,20 +55,15 @@
   </link>
   <link name="link3">
-    <collision>
-      <origin xyz="0 0 0.45" rpy="0 0 0"/>
-      <geometry>
-        <box size="0.1 0.1 1"/>
-      </geometry>
-      <material name="blue"/>
+    <collision name="collision">
+      <origin xyz="0.5 0 0" rpy="0 0 0"/>
+      <geometry> <box size="0.9 0.1 0.1"/> </geometry>
     </collision>
-    <visual>
-      <origin xyz="0 0 0.45" rpy="0 0 0"/>
-      <geometry>
-        <box size="0.1 0.1 1"/>
-      </geometry>
+    <visual name="visual">
+      <origin xyz="0.5 0 0" rpy="0 0 0"/>
+      <geometry> <box size="1 0.1 0.1"/> </geometry>
       <material name="blue"/>
     </visual>
     <inertial>
-      <origin xyz="0 0 1.5" rpy="0 0 0"/>
+      <origin xyz="0.5 0 0" rpy="0 0 0"/>
       <mass value="1"/>
       <inertia
@@ -88,23 +73,19 @@
     </inertial>
   </link>
-  <gazebo reference="link3">
-    <mu1>0.2</mu1>
-    <mu2>0.2</mu2>
-  </gazebo>
   <joint name="fixed" type="fixed">
     <parent link="world"/>
     <child link="link1"/>
-    <!--origin xyz="0 0 1" rpy="${PI} 0 0"/-->
+    <origin xyz="0 0 1" rpy="${PI} 0 0"/>
   </joint>
   <joint name="joint1" type="continuous">
     <parent link="link1"/>
     <child link="link2"/>
-    <origin xyz="0 0.1 0.9" rpy="0 0 0"/>
-    <axis xyz="0 1 0"/>
+    <origin xyz="1 0 0" rpy="0 0 0"/>
+    <axis xyz="0 0 1"/>
   </joint>
   <joint name="joint2" type="continuous">
     <parent link="link2"/>
     <child link="link3"/>
-    <origin xyz="0 0.1 0.9" rpy="0 0 0"/>
+    <origin xyz="1 0 0" rpy="0 0 0"/>
     <axis xyz="0 1 0"/>
   </joint>
