Commit message: removing error case when sim type is not given

File: gazebo_ros_control_examples/models/rr_manipulator_custom_interface.urdf.xacro (robot description, xacro)
@@ -7,8 +7,7 @@
   <gazebo>
     <plugin name="ros_control" filename="libgazebo_ros_control_plugin.so">
-      <robotNamespace>rr/ros_control</robotNamespace>
+      <ns>rr/ros_control</ns>
+      <robotSimType>gazebo_ros_control_examples/RobotSimRR</robotSimType>
       <controlPeriod>0.001</controlPeriod>
-      <joint>joint1</joint>
-      <joint>joint2</joint>
     </plugin>
   </gazebo>
