Commit message: working camera added

File: gazebo_plugins/test/diff_drive/xacro/laser/hokuyo.xacro (robot description, xacro)
@@ -1,63 +1,63 @@
 <?xml version="1.0"?>
 <robot xmlns:xacro="http://www.ros.org/wiki/xacro">
-  <!-- Front Laser -->
-  <xacro:macro name="front_laser" params="xyz rpy">
-	  <joint name="front_laser_joint" type="fixed">
-		<axis xyz="0 0 1" />
-		<origin xyz="${xyz}" rpy="${rpy}"/>
-		<parent link="base_link"/>
-		<child link="front_laser"/>
-	  </joint>
-	  <link name="front_laser">
-		<collision>
-		  <origin xyz="0 0 0" rpy="0 0 0"/>
-		  <geometry>
-			<box size="0.1 0.1 0.1"/>
-		  </geometry>
-		</collision>
-		<visual>
-		  <origin xyz="0 0 0" rpy="0 0 0"/>
-		  <geometry>
-			<mesh filename="package://gazebo_plugins/test/diff_drive/meshes/laser/hokuyo.dae"/>
-		  </geometry>
-		</visual>
-		<inertial>
-		  <mass value="1e-5" />
-		  <origin xyz="0 0 0" rpy="0 0 0"/>
-		  <inertia ixx="1e-6" ixy="0" ixz="0" iyy="1e-6" iyz="0" izz="1e-6" />
-		</inertial>
-	  </link>
-	  <gazebo reference="front_laser">
-		  <sensor name="laser" type="ray">
-		  <pose>0 0 0 0 0 0</pose>
-			<ray>
-			  <scan>
-				<horizontal>
-				  <!-- The URG-04LX-UG01  has  683 steps with 0.35139 Degree resolution -->
-				  <resolution>1</resolution>
-				  <max_angle>2.0944</max_angle> <!-- 120 Degree -->
-				  <min_angle>-2.0944</min_angle> <!-- -120 Degree -->
-				  <samples>683</samples>
-				</horizontal>
-			  </scan>
-			  <range>
-				<min>0.08</min>
-				<max>5</max>
-				<resolution>0.01</resolution>
-			  </range>
-			</ray>
-			<plugin name="laser" filename="libgazebo_ros_laser.so" >
-        <robotNamespace></robotNamespace>
-			  <topicName>front_laser/scan</topicName>
-			  <frameName>front_laser</frameName>
-			</plugin>
-			<!--
-			<plugin name="laser" filename="libRayPlugin.so" />
-			-->
-			<always_on>1</always_on>
-			<update_rate>30</update_rate>
-			<visualize>true</visualize>
-		  </sensor>
-	  </gazebo>
-  </xacro:macro>
+<!-- Front Laser -->
+<xacro:macro name="front_laser" params="xyz rpy">
+  <joint name="front_laser_joint" type="fixed">
+      <axis xyz="0 0 1" />
+      <origin xyz="${xyz}" rpy="${rpy}"/>
+      <parent link="base_link"/>
+      <child link="front_laser"/>
+    </joint>
+    <link name="front_laser">
+      <collision>
+        <origin xyz="0 0 0" rpy="0 0 0"/>
+        <geometry>
+          <box size="0.1 0.1 0.1"/>
+        </geometry>
+      </collision>
+      <visual>
+        <origin xyz="0 0 0" rpy="0 0 0"/>
+        <geometry>
+          <mesh filename="package://gazebo_plugins/test/diff_drive/meshes/laser/hokuyo.dae"/>
+        </geometry>
+      </visual>
+      <inertial>
+        <mass value="1e-5" />
+        <origin xyz="0 0 0" rpy="0 0 0"/>
+        <inertia ixx="1e-6" ixy="0" ixz="0" iyy="1e-6" iyz="0" izz="1e-6" />
+      </inertial>
+    </link>
+    <gazebo reference="front_laser">
+        <sensor name="laser" type="ray">
+        <pose>0 0 0 0 0 0</pose>
+          <ray>
+            <scan>
+              <horizontal>
+                <!-- The URG-04LX-UG01  has  683 steps with 0.35139 Degree resolution -->
+                <resolution>1</resolution>
+                <max_angle>2.0944</max_angle> <!-- 120 Degree -->
+                <min_angle>-2.0944</min_angle> <!-- -120 Degree -->
+                <samples>683</samples>
+              </horizontal>
+            </scan>
+            <range>
+              <min>0.08</min>
+              <max>5</max>
+              <resolution>0.01</resolution>
+            </range>
+          </ray>
+          <plugin name="laser" filename="libgazebo_ros_laser.so" >
+            <robotNamespace></robotNamespace>
+            <topicName>front_laser/scan</topicName>
+            <frameName>front_laser</frameName>
+          </plugin>
+          <!--
+          <plugin name="laser" filename="libRayPlugin.so" />
+          -->
+          <always_on>1</always_on>
+          <update_rate>30</update_rate>
+          <visualize>true</visualize>
+        </sensor>
+    </gazebo>
+</xacro:macro>
 </robot>

File: gazebo_plugins/test/diff_drive/xacro/p3dx/pioneer3dx.xacro (robot description, xacro)
@@ -1,7 +1,11 @@
 <?xml version="1.0"?>
 <robot xmlns:xacro="http://www.ros.org/wiki/xacro" name="pioneer3dx">
+  <!-- Import Rviz colors -->
+  <xacro:include filename="$(find gazebo_plugins)/test/diff_drive/xacro/materials.xacro" />
   <xacro:include filename="$(find gazebo_plugins)/test/diff_drive/xacro/p3dx/pioneer3dx_body.xacro"/>
   <xacro:pioneer3dx_body />
   <xacro:include filename="$(find gazebo_plugins)/test/diff_drive/xacro/laser/hokuyo.xacro"/>
-  <xacro:front_laser xyz="0.16 0 0.1" rpy="0 0 0"/>
+  <xacro:front_laser xyz="0.16 0 0.1" rpy="0 0 0" />
+  <xacro:include filename="$(find gazebo_plugins)/test/diff_drive/xacro/camera/camera.xacro"/>
+  <xacro:cam_front xyz="0 0 0.5" rpy="0 0 0" />
 </robot>
