Commit message: gazebo test model pionneer 3dx updated with xacro path variables

File: gazebo_plugins/test/multi_robot_scenario/xacro/laser/hokuyo.xacro (robot description, xacro)
@@ -2,5 +2,5 @@
 <robot xmlns:xacro="http://www.ros.org/wiki/xacro">
 <!-- Front Laser -->
-<xacro:macro name="front_laser" params="xyz rpy">
+<xacro:macro name="front_laser" params="xyz rpy meshes" >
   <joint name="front_laser_joint" type="fixed">
       <axis xyz="0 0 1" />

File: gazebo_plugins/test/multi_robot_scenario/xacro/p3dx/battery_block.xacro (robot description, xacro)
@@ -1,5 +1,4 @@
 <?xml version="1.0"?>
-<robot
-  xmlns:xacro="http://ros.org/wiki/xacro">
+<robot xmlns:xacro="http://ros.org/wiki/xacro">
   <property name="M_PI" value="3.1415926535897931" />
   <xacro:macro name="battery_block" params="name parent x y z mass">

File: gazebo_plugins/test/multi_robot_scenario/xacro/p3dx/inertia_tensors.xacro (robot description, xacro)
@@ -3,6 +3,5 @@
   see https://github.com/uos/uos_tools/blob/fuerte/uos_common_urdf/common.xacro and
   see http://answers.gazebosim.org/question/4372/the-inertia-matrix-explained/ -->
-<robot
-  xmlns:xacro="http://ros.org/wiki/xacro">
+<robot xmlns:xacro="http://ros.org/wiki/xacro">
   <property name="M_PI" value="3.1415926535897931" />
   <!-- see https://secure.wikimedia.org/wikipedia/en/wiki/List_of_moment_of_inertia_tensors -->

File: gazebo_plugins/test/multi_robot_scenario/xacro/p3dx/pioneer3dx.xacro (robot description, xacro)
@@ -1,10 +1,11 @@
 <?xml version="1.0"?>
-<robot xmlns:xacro="http://www.ros.org/wiki/xacro" name="pioneer3dx">
+<robot xmlns:xacro="http://www.ros.org/wiki/xacro" name="pioneer3dx" >
   <!-- Import Rviz colors -->
   <xacro:include filename="$(find gazebo_plugins)/test/multi_robot_scenario/xacro/materials.xacro" />
+  <!-- Import robot -->
   <xacro:include filename="$(find gazebo_plugins)/test/multi_robot_scenario/xacro/p3dx/pioneer3dx_body.xacro"/>
-  <xacro:pioneer3dx_body />
+  <xacro:pioneer3dx_body meshes="package://gazebo_plugins/test/multi_robot_scenario/meshes/p3dx"/>
   <xacro:include filename="$(find gazebo_plugins)/test/multi_robot_scenario/xacro/laser/hokuyo.xacro"/>
-  <xacro:front_laser xyz="0.16 0 0.1" rpy="0 0 0" />
+  <xacro:front_laser xyz="0.16 0 0.1" rpy="0 0 0" meshes="package://gazebo_plugins/test/multi_robot_scenario/meshes/laser"/>
   <xacro:include filename="$(find gazebo_plugins)/test/multi_robot_scenario/xacro/camera/camera.xacro"/>
   <xacro:cam_front xyz="0 0 0.5" rpy="0 0 0" />

File: gazebo_plugins/test/multi_robot_scenario/xacro/p3dx/pioneer3dx_body.xacro (robot description, xacro)
@@ -1,132 +1,28 @@
 <?xml version="1.0"?>
 <robot xmlns:xacro="http://www.ros.org/wiki/xacro">
-  <!-- Import all Gazebo-customization elements, including Gazebo colors -->
-  <xacro:include filename="$(find gazebo_plugins)/test/multi_robot_scenario/xacro/p3dx/inertia_tensors.xacro"/>
-  <xacro:include filename="$(find gazebo_plugins)/test/multi_robot_scenario/xacro/p3dx/battery_block.xacro"/>
-  <xacro:include filename="$(find gazebo_plugins)/test/multi_robot_scenario/xacro/p3dx/pioneer3dx_wheel.xacro"/>
-  <xacro:include filename="$(find gazebo_plugins)/test/multi_robot_scenario/xacro/p3dx/pioneer3dx_swivel.xacro"/>
-  <xacro:macro name="pioneer3dx_body" params="">
-  <!-- base_link -->
-  <link name="base_link"/>
-  <gazebo reference="base_link">
-    <material value="Gazebo/Red"/>
-  </gazebo>
-  <!-- Chassis -->
-  <joint name="base_chassis_joint" type="fixed">
-    <origin xyz="0 0 0" rpy="0 0 0"/>
-    <parent link="base_link"/>
-    <child link="chassis"/>
-  </joint>
-  <link name="chassis">
-    <visual name="chassis_visual">
-      <origin xyz="-0.045 0 0.148" rpy="0 0 0"/>
-      <geometry name="pioneer_geom">
-        <mesh filename="package://v4r_gazebo/meshes/p3dx_meshes/chassis.stl"/>
-      </geometry>
-      <material name="ChassisRed">
-        <color rgba="0.851 0.0 0.0 1.0"/>
-      </material>
-    </visual>
-    <collision>
-      <origin xyz="-0.045 0 0.148" rpy="0 0 0"/>
-      <geometry>
-        <mesh filename="package://v4r_gazebo/meshes/p3dx_meshes/chassis.stl"/>
-      </geometry>
-    </collision>
-    <xacro:box_inertial x="0.36" y="0.26"  z="0.18" mass="9.0" />
-  </link>
-  <gazebo reference="chassis">
-    <material value="Gazebo/Red"/>
-  </gazebo>
-  <!-- Akku0 -->
-  <xacro:battery_block name="accu0" parent="chassis" x="-0.14" y="0.00"  z="0.13" mass="2.5" />
-  <!-- Top -->
-  <joint name="chassis_top_joint" type="fixed">
-    <origin xyz="-0.045 0 0.234" rpy="0 0 0"/>
-    <parent link="chassis"/>
-    <child link="top_plate"/>
-  </joint>
-  <link name="top_plate">
-    <visual>
-      <origin xyz="0 0 0" rpy="0 0 0"/>
-      <geometry name="top_geom">
-        <mesh filename="package://v4r_gazebo/meshes/p3dx_meshes/top.stl"/>
-      </geometry>
-      <material name="TopBlack">
-        <color rgba="0.038 0.038 0.038 1.0"/>
-      </material>
-    </visual>
-    <collision>
-    <origin xyz="0.0 0 0.0" rpy="0 0 0"/>
-      <geometry>
-        <mesh filename="package://v4r_gazebo/meshes/p3dx_meshes/top.stl"/>
-      </geometry>
-    </collision>
-    <xacro:box_inertial x="0.445" y="0.38"  z="0.01" mass="1.0" />
-  </link>
-  <gazebo reference="top_plate">
-    <material value="Gazebo/Black"/>
-  </gazebo>
-  <!-- Wheels -->
-  <xacro:pioneer_swivel parent="chassis"  xyz="-0.185 0 0.055" rpy="0 0 0" />
-  <xacro:pioneer_wheel side="right" parent="chassis"  xyz="0  0.15 0.09" rpy="0 0 0" radius="0.09"/>
-  <xacro:pioneer_wheel side="left"  parent="chassis"  xyz="0 -0.15 0.09" rpy="0 0 0" radius="0.09"/>
-  <!-- Front Sonar -->
-  <joint name="base_front_joint" type="fixed">
-    <origin xyz="0.109 0 0.209" rpy="0 0 0"/>
-    <parent link="base_link"/>
-    <child link="front_sonar"/>
-  </joint>
-  <link name="front_sonar">
-    <inertial>
-      <mass value="0.0001"/>
-      <origin xyz="0 0 0"/>
-      <inertia ixx="1" ixy="0" ixz="0" iyy="1" iyz="0" izz="1"/>
-    </inertial>
-    <visual name="front_sonar_vis">
-      <origin xyz="0 0 0" rpy="0 0 0"/>
-      <geometry name="pioneer_geom">
-        <mesh filename="package://v4r_gazebo/meshes/p3dx_meshes/back_sonar.stl"/>
-      </geometry>
-      <material name="SonarYellow">
-        <color rgba="0.715 0.583 0.210 1.0"/>
-      </material>
-    </visual>
-    <collision>
-      <origin xyz="0 0 0" rpy="0 0 0"/>
-      <geometry>
-        <box size="0 0 0"/>
-      </geometry>
-    </collision>
-  </link>
-  <gazebo reference="front_sonar">
-    <material value="Gazebo/Yellow"/>
-  </gazebo>
-  <gazebo>
-      <plugin name="joint_state_publisher" filename="libgazebo_ros_joint_state_publisher.so">
-        <robotNamespace></robotNamespace>
-        <jointName>chassis_swivel_joint, swivel_wheel_joint, left_hub_joint, right_hub_joint</jointName>
-        <updateRate>10.0</updateRate>
-        <alwaysOn>true</alwaysOn>
-      </plugin>
-  </gazebo>
-    <gazebo>
-        <plugin name="differential_drive_controller" filename="libgazebo_ros_diff_drive.so">
-            <robotNamespace></robotNamespace>
-            <publishWheelTF>false</publishWheelTF>
-            <publishWheelJointState>true</publishWheelJointState>
-            <alwaysOn>true</alwaysOn>
-            <leftJoint>left_hub_joint</leftJoint>
-            <rightJoint>right_hub_joint</rightJoint>
-            <wheelSeparation>0.5380</wheelSeparation>
-            <wheelDiameter>0.18</wheelDiameter>
-            <torque>20</torque>
-            <commandTopic>cmd_vel</commandTopic>
-            <odometryTopic>odom</odometryTopic>
-            <odometryFrame>odom</odometryFrame>
-            <robotBaseFrame>base_link</robotBaseFrame>
-            <updateRate>100.0</updateRate>
-        </plugin>
-    </gazebo>
+  <xacro:include filename="inertia_tensors.xacro"/>
+  <xacro:include filename="pioneer3dx_chassis.xacro"/>
+  <xacro:include filename="battery_block.xacro"/>
+  <xacro:include filename="pioneer3dx_wheel.xacro"/>
+  <xacro:include filename="pioneer3dx_swivel.xacro"/>
+  <xacro:include filename="pioneer3dx_sonar.xacro"/>
+  <xacro:include filename="pioneer3dx_plugins.xacro"/>
+  <xacro:macro name="pioneer3dx_body" params="meshes">
+    <!-- base_link -->
+    <link name="base_link"/>
+    <!-- Chassis -->
+    <xacro:pioneer_chassis name="chassis" parent="base_link" xyz="0 0 0" rpy="0 0 0"  meshes="${meshes}"/>
+    <!-- Front Sonar -->
+    <xacro:pioneer_sonar name="sonar" parent="chassis" xyz="0.109 0 0.209" rpy="0 0 0"  meshes="${meshes}"/>
+    <!-- Akku0 -->
+    <xacro:battery_block name="battery0" parent="chassis" x="-0.14" y="0.00"  z="0.13" mass="2.5" />
+    <!-- Wheels -->
+    <xacro:pioneer_wheel side="right" parent="chassis"  xyz="0  0.15 0.09" rpy="0 0 0" radius="0.09" meshes="${meshes}"/>
+    <xacro:pioneer_wheel side="left"  parent="chassis"  xyz="0 -0.15 0.09" rpy="0 0 0" radius="0.09" meshes="${meshes}"/>
+    <xacro:pioneer_swivel parent="chassis"  xyz="-0.185 0 0.055" rpy="0 0 0" meshes="${meshes}"/>
+    <!-- Motor plugin -->
+    <xacro:pioneer3dx_diff_drive />
+    <!-- Joints plugin -->
+    <xacro:pioneer3dx_joints_state_publisher />
   </xacro:macro>
 </robot>

File: gazebo_plugins/test/multi_robot_scenario/xacro/p3dx/pioneer3dx_swivel.xacro (robot description, xacro)
@@ -1,7 +1,6 @@
 <?xml version="1.0"?>
-<robot
-  xmlns:xacro="http://ros.org/wiki/xacro">
+<robot xmlns:xacro="http://ros.org/wiki/xacro">
   <property name="M_PI" value="3.1415926535897931" />
-  <xacro:macro name="pioneer_swivel" params="parent xyz rpy">
+  <xacro:macro name="pioneer_swivel" params="parent xyz rpy meshes">
   <!-- Swivel -->
   <joint name="chassis_swivel_joint" type="continuous">
@@ -23,5 +22,5 @@
       <origin xyz="0 0 0" rpy="0 0 0"/>
       <geometry name="pioneer_geom">
-        <mesh filename="package://v4r_gazebo/meshes/p3dx_meshes/swivel.stl"/>
+        <mesh filename="${meshes}/swivel.stl"/>
       </geometry>
       <material name="swivel">
@@ -58,5 +57,5 @@
       <origin xyz="0 0 0" rpy="0 0 0"/>
       <geometry name="pioneer_geom">
-        <mesh filename="package://v4r_gazebo/meshes/p3dx_meshes/center_wheel.stl"/>
+        <mesh filename="${meshes}/center_wheel.stl"/>
       </geometry>
       <material name="WheelBlack">
@@ -67,5 +66,5 @@
       <origin xyz="0 0 0" rpy="${-3.1415927/2.0} 0 0"/>
       <geometry>
-        <!--<mesh filename="package://v4r_gazebo/meshes/p3dx_meshes/center_wheel.stl"/>-->
+        <!--<mesh filename="${meshes}/center_wheel.stl"/>-->
         <cylinder radius="0.0375" length="0.01"/>
       </geometry>
@@ -90,5 +89,5 @@
       <origin xyz="0 0 0" rpy="0 0 0"/>
       <geometry name="pioneer_geom">
-        <mesh filename="package://v4r_gazebo/meshes/p3dx_meshes/center_hubcap.stl"/>
+        <mesh filename="${meshes}/center_hubcap.stl"/>
       </geometry>
       <material name="swivel">

File: gazebo_plugins/test/multi_robot_scenario/xacro/p3dx/pioneer3dx_wheel.xacro (robot description, xacro)
@@ -3,5 +3,5 @@
   xmlns:xacro="http://ros.org/wiki/xacro">
   <property name="M_PI" value="3.1415926535897931" />
-  <xacro:macro name="pioneer_wheel" params="side parent xyz rpy radius">
+  <xacro:macro name="pioneer_wheel" params="side parent xyz rpy radius meshes">
   <!-- Hubcap -->
   <joint name="${side}_hub_joint" type="continuous">
@@ -20,5 +20,5 @@
       <origin xyz="0 0 0" rpy="0 0 0"/>
       <geometry name="pioneer_geom">
-        <mesh filename="package://v4r_gazebo/meshes/p3dx_meshes/${side}_hubcap.stl"/>
+        <mesh filename="${meshes}/${side}_hubcap.stl"/>
       </geometry>
       <material name="HubcapYellow">
@@ -52,5 +52,5 @@
       <origin xyz="0 0 0" rpy="0 0 0"/>
       <geometry name="pioneer_geom">
-        <mesh filename="package://v4r_gazebo/meshes/p3dx_meshes/${side}_wheel.stl"/>
+        <mesh filename="${meshes}/${side}_wheel.stl"/>
       </geometry>
       <material name="WheelBlack">
@@ -61,5 +61,5 @@
       <origin xyz="0 0 0" rpy="${-3.1415927/2} 0 0"/>
       <geometry>
-        <!--<mesh filename="package://v4r_gazebo/meshes/p3dx_meshes/${side}_wheel.stl"/>-->
+        <!--<mesh filename="${meshes}/${side}_wheel.stl"/>-->
         <cylinder radius="${radius}" length="0.01"/>
       </geometry>
