Commit message: fixed links related to changed name

File: gazebo_plugins/test/multi_robot_scenario/xacro/camera/camera.xacro (robot description, xacro)
@@ -21,5 +21,5 @@
         <cylinder radius="0.03" length="0.1"/>
       </geometry>
-      <material name="orange"/>
+      <material name="grey"/>
     </visual>
     <collision>
@@ -31,5 +31,5 @@
   </link>
   <gazebo reference="front_camera">
-    <material value="Gazebo/Orange"/>
+    <material value="Gazebo/grey"/>
   </gazebo>
   <gazebo reference="front_camera">

File: gazebo_plugins/test/multi_robot_scenario/xacro/laser/hokuyo.xacro (robot description, xacro)
@@ -19,5 +19,5 @@
         <origin xyz="0 0 0" rpy="0 0 0"/>
         <geometry>
-          <mesh filename="package://gazebo_plugins/test/diff_drive/meshes/laser/hokuyo.dae"/>
+          <mesh filename="package://gazebo_plugins/test/multi_robot_scenario/meshes/laser/hokuyo.dae"/>
         </geometry>
       </visual>

File: gazebo_plugins/test/multi_robot_scenario/xacro/p3dx/pioneer3dx.xacro (robot description, xacro)
@@ -2,10 +2,10 @@
 <robot xmlns:xacro="http://www.ros.org/wiki/xacro" name="pioneer3dx">
   <!-- Import Rviz colors -->
-  <xacro:include filename="$(find gazebo_plugins)/test/diff_drive/xacro/materials.xacro" />
-  <xacro:include filename="$(find gazebo_plugins)/test/diff_drive/xacro/p3dx/pioneer3dx_body.xacro"/>
+  <xacro:include filename="$(find gazebo_plugins)/test/multi_robot_scenario/xacro/materials.xacro" />
+  <xacro:include filename="$(find gazebo_plugins)/test/multi_robot_scenario/xacro/p3dx/pioneer3dx_body.xacro"/>
   <xacro:pioneer3dx_body />
-  <xacro:include filename="$(find gazebo_plugins)/test/diff_drive/xacro/laser/hokuyo.xacro"/>
+  <xacro:include filename="$(find gazebo_plugins)/test/multi_robot_scenario/xacro/laser/hokuyo.xacro"/>
   <xacro:front_laser xyz="0.16 0 0.1" rpy="0 0 0" />
-  <xacro:include filename="$(find gazebo_plugins)/test/diff_drive/xacro/camera/camera.xacro"/>
+  <xacro:include filename="$(find gazebo_plugins)/test/multi_robot_scenario/xacro/camera/camera.xacro"/>
   <xacro:cam_front xyz="0 0 0.5" rpy="0 0 0" />
 </robot>

File: gazebo_plugins/test/multi_robot_scenario/xacro/p3dx/pioneer3dx_body.xacro (robot description, xacro)
@@ -18,5 +18,5 @@
       <origin xyz="-0.045 0 0.148" rpy="0 0 0"/>
       <geometry name="pioneer_geom">
-        <mesh filename="package://gazebo_plugins/test/diff_drive/meshes/p3dx/chassis.stl"/>
+        <mesh filename="package://gazebo_plugins/test/multi_robot_scenario/meshes/p3dx/chassis.stl"/>
       </geometry>
       <material name="ChassisRed">
@@ -27,5 +27,5 @@
       <origin xyz="-0.045 0 0.148" rpy="0 0 0"/>
       <geometry>
-        <mesh filename="package://gazebo_plugins/test/diff_drive/meshes/p3dx/chassis.stl"/>
+        <mesh filename="package://gazebo_plugins/test/multi_robot_scenario/meshes/p3dx/chassis.stl"/>
       </geometry>
     </collision>
@@ -54,5 +54,5 @@
       <origin xyz="0 0 0" rpy="0 0 0"/>
       <geometry name="top_geom">
-        <mesh filename="package://gazebo_plugins/test/diff_drive/meshes/p3dx/top.stl"/>
+        <mesh filename="package://gazebo_plugins/test/multi_robot_scenario/meshes/p3dx/top.stl"/>
       </geometry>
       <material name="TopBlack">
@@ -84,5 +84,5 @@
       <origin xyz="0 0 0" rpy="0 0 0"/>
       <geometry name="pioneer_geom">
-        <mesh filename="package://gazebo_plugins/test/diff_drive/meshes/p3dx/swivel.stl"/>
+        <mesh filename="package://gazebo_plugins/test/multi_robot_scenario/meshes/p3dx/swivel.stl"/>
       </geometry>
       <material name="swivel">
@@ -119,5 +119,5 @@
       <origin xyz="0 0 0" rpy="0 0 0"/>
       <geometry name="pioneer_geom">
-        <mesh filename="package://gazebo_plugins/test/diff_drive/meshes/p3dx/center_wheel.stl"/>
+        <mesh filename="package://gazebo_plugins/test/multi_robot_scenario/meshes/p3dx/center_wheel.stl"/>
       </geometry>
       <material name="WheelBlack">
@@ -128,5 +128,5 @@
       <origin xyz="0 0 0" rpy="${-3.1415927/2.0} 0 0"/>
       <geometry>
-        <!--<mesh filename="package://gazebo_plugins/test/diff_drive/meshes/p3dx/center_wheel.stl"/>-->
+        <!--<mesh filename="package://gazebo_plugins/test/multi_robot_scenario/meshes/p3dx/center_wheel.stl"/>-->
         <cylinder radius="0.0375" length="0.01"/>
       </geometry>
@@ -151,5 +151,5 @@
       <origin xyz="0 0 0" rpy="0 0 0"/>
       <geometry name="pioneer_geom">
-        <mesh filename="package://gazebo_plugins/test/diff_drive/meshes/p3dx/center_hubcap.stl"/>
+        <mesh filename="package://gazebo_plugins/test/multi_robot_scenario/meshes/p3dx/center_hubcap.stl"/>
       </geometry>
       <material name="swivel">
@@ -183,5 +183,5 @@
       <origin xyz="0 0 0" rpy="0 0 0"/>
       <geometry name="pioneer_geom">
-        <mesh filename="package://gazebo_plugins/test/diff_drive/meshes/p3dx/right_hubcap.stl"/>
+        <mesh filename="package://gazebo_plugins/test/multi_robot_scenario/meshes/p3dx/right_hubcap.stl"/>
       </geometry>
       <material name="HubcapYellow">
@@ -215,5 +215,5 @@
       <origin xyz="0 0 0" rpy="0 0 0"/>
       <geometry name="pioneer_geom">
-        <mesh filename="package://gazebo_plugins/test/diff_drive/meshes/p3dx/right_wheel.stl"/>
+        <mesh filename="package://gazebo_plugins/test/multi_robot_scenario/meshes/p3dx/right_wheel.stl"/>
       </geometry>
       <material name="WheelBlack">
@@ -224,5 +224,5 @@
       <origin xyz="0 0 0" rpy="${-3.1415927/2} 0 0"/>
       <geometry>
-        <!--<mesh filename="package://gazebo_plugins/test/diff_drive/meshes/p3dx/${suffix}_wheel.stl"/>-->
+        <!--<mesh filename="package://gazebo_plugins/test/multi_robot_scenario/meshes/p3dx/${suffix}_wheel.stl"/>-->
         <cylinder radius="0.09" length="0.01"/>
       </geometry>
@@ -248,5 +248,5 @@
       <origin xyz="0 0 0" rpy="0 0 0"/>
       <geometry name="pioneer_geom">
-        <mesh filename="package://gazebo_plugins/test/diff_drive/meshes/p3dx/left_hubcap.stl"/>
+        <mesh filename="package://gazebo_plugins/test/multi_robot_scenario/meshes/p3dx/left_hubcap.stl"/>
       </geometry>
       <material name="HubcapYellow">
@@ -280,5 +280,5 @@
       <origin xyz="0 0 0" rpy="0 0 0"/>
       <geometry name="pioneer_geom">
-        <mesh filename="package://gazebo_plugins/test/diff_drive/meshes/p3dx/left_wheel.stl"/>
+        <mesh filename="package://gazebo_plugins/test/multi_robot_scenario/meshes/p3dx/left_wheel.stl"/>
       </geometry>
       <material name="WheelBlack">
@@ -289,5 +289,5 @@
       <origin xyz="0 0 0" rpy="${-3.1415927/2} 0 0"/>
       <geometry>
-        <!--<mesh filename="package://gazebo_plugins/test/diff_drive/meshes/p3dx/${suffix}_wheel.stl"/>-->
+        <!--<mesh filename="package://gazebo_plugins/test/multi_robot_scenario/meshes/p3dx/${suffix}_wheel.stl"/>-->
         <cylinder radius="0.09" length="0.01"/>
       </geometry>
@@ -312,5 +312,5 @@
       <origin xyz="0 0 0" rpy="0 0 0"/>
       <geometry name="pioneer_geom">
-        <mesh filename="package://gazebo_plugins/test/diff_drive/meshes/p3dx/back_sonar.stl"/>
+        <mesh filename="package://gazebo_plugins/test/multi_robot_scenario/meshes/p3dx/back_sonar.stl"/>
       </geometry>
       <material name="SonarYellow">

Commit message: fixed camera to work with workspaces

File: gazebo_plugins/test/multi_robot_scenario/xacro/camera/camera.xacro (robot description, xacro)
@@ -31,5 +31,5 @@
   </link>
   <gazebo reference="front_camera">
-    <material value="Gazebo/grey"/>
+    <material value="Gazebo/Grey"/>
   </gazebo>
   <gazebo reference="front_camera">
@@ -57,4 +57,5 @@
       </camera>
       <plugin name="camera_controller" filename="libgazebo_ros_camera.so">
+        <robotNamespace>rr</robotNamespace>
         <alwaysOn>true</alwaysOn>
         <updateRate>0.0</updateRate>

Commit message: minor fixes on relative paths in xacro for pioneer robot

File: gazebo_plugins/test/multi_robot_scenario/xacro/camera/camera.xacro (robot description, xacro)
@@ -2,13 +2,13 @@
 <robot xmlns:xacro="http://www.ros.org/wiki/xacro">
 <!-- Camera -->
-<xacro:macro name="cam_front" params="xyz rpy">
-  <joint name="base_front_camera_joint" type="fixed">
-          <axis xyz="0 0 1" />
-          <origin xyz="${xyz}" rpy="${rpy}"/>
-          <parent link="base_link"/>
-          <child link="front_camera"/>
+<xacro:macro name="cam" params="name parent xyz rpy">
+  <joint name="${parent}_${name}_joint" type="fixed">
+      <axis xyz="0 0 1" />
+      <origin xyz="${xyz}" rpy="${rpy}"/>
+      <parent link="${parent}"/>
+      <child link="${name}"/>
   </joint>
   <!-- Camera -->
-  <link name="front_camera">
+  <link name="${name}">
     <inertial>
       <mass value="1e-5" />
@@ -30,8 +30,8 @@
     </collision>
   </link>
-  <gazebo reference="front_camera">
+  <gazebo reference="${name}">
     <material value="Gazebo/Grey"/>
   </gazebo>
-  <gazebo reference="front_camera">
+  <gazebo reference="${name}">
     <sensor type="camera" name="camera1">
       <update_rate>30.0</update_rate>
@@ -60,8 +60,8 @@
         <alwaysOn>true</alwaysOn>
         <updateRate>0.0</updateRate>
-        <cameraName>camera</cameraName>
+        <cameraName>${name}</cameraName>
         <imageTopicName>image_raw</imageTopicName>
         <cameraInfoTopicName>camera_info</cameraInfoTopicName>
-        <frameName>front_camera</frameName>
+        <frameName>${name}</frameName>
         <hackBaseline>0.07</hackBaseline>
         <distortionK1>0.0</distortionK1>

File: gazebo_plugins/test/multi_robot_scenario/xacro/laser/hokuyo.xacro (robot description, xacro)
@@ -2,12 +2,12 @@
 <robot xmlns:xacro="http://www.ros.org/wiki/xacro">
 <!-- Front Laser -->
-<xacro:macro name="front_laser" params="xyz rpy meshes" >
-  <joint name="front_laser_joint" type="fixed">
+<xacro:macro name="laser" params="name parent xyz rpy meshes" >
+  <joint name="${parent}_${name}_joint" type="fixed">
       <axis xyz="0 0 1" />
       <origin xyz="${xyz}" rpy="${rpy}"/>
-      <parent link="base_link"/>
-      <child link="front_laser"/>
+      <parent link="${parent}"/>
+      <child link="${name}"/>
     </joint>
-    <link name="front_laser">
+    <link name="${name}">
       <collision>
         <origin xyz="0 0 0" rpy="0 0 0"/>
@@ -19,5 +19,5 @@
         <origin xyz="0 0 0" rpy="0 0 0"/>
         <geometry>
-          <mesh filename="package://gazebo_plugins/test/multi_robot_scenario/meshes/laser/hokuyo.dae"/>
+          <mesh filename="${meshes}/hokuyo.dae"/>
         </geometry>
       </visual>
@@ -28,5 +28,5 @@
       </inertial>
     </link>
-    <gazebo reference="front_laser">
+    <gazebo reference="${name}">
         <sensor name="laser" type="ray">
         <pose>0 0 0 0 0 0</pose>
@@ -49,6 +49,6 @@
           <plugin name="laser" filename="libgazebo_ros_laser.so" >
             <robotNamespace></robotNamespace>
-            <topicName>front_laser/scan</topicName>
-            <frameName>front_laser</frameName>
+            <topicName>${name}/scan</topicName>
+            <frameName>${name}</frameName>
           </plugin>
           <!--

File: gazebo_plugins/test/multi_robot_scenario/xacro/p3dx/pioneer3dx.xacro (robot description, xacro)
@@ -5,8 +5,8 @@
   <!-- Import robot -->
   <xacro:include filename="$(find gazebo_plugins)/test/multi_robot_scenario/xacro/p3dx/pioneer3dx_body.xacro"/>
-  <xacro:pioneer3dx_body meshes="package://gazebo_plugins/test/multi_robot_scenario/meshes/p3dx"/>
+  <xacro:pioneer3dx_body name="chassis" parent="base_link" meshes="package://gazebo_plugins/test/multi_robot_scenario/meshes/p3dx"/>
   <xacro:include filename="$(find gazebo_plugins)/test/multi_robot_scenario/xacro/laser/hokuyo.xacro"/>
-  <xacro:front_laser xyz="0.16 0 0.1" rpy="0 0 0" meshes="package://gazebo_plugins/test/multi_robot_scenario/meshes/laser"/>
+  <xacro:laser name="front_laser" parent="chassis" xyz="0.16 0 0.1" rpy="0 0 0" meshes="package://gazebo_plugins/test/multi_robot_scenario/meshes/laser"/>
   <xacro:include filename="$(find gazebo_plugins)/test/multi_robot_scenario/xacro/camera/camera.xacro"/>
-  <xacro:cam_front xyz="0 0 0.5" rpy="0 0 0" />
+  <xacro:cam name="front_camera" parent="chassis" xyz="0 0 0.5" rpy="0 0 0" />
 </robot>

File: gazebo_plugins/test/multi_robot_scenario/xacro/p3dx/pioneer3dx_body.xacro (robot description, xacro)
@@ -8,17 +8,17 @@
   <xacro:include filename="pioneer3dx_sonar.xacro"/>
   <xacro:include filename="pioneer3dx_plugins.xacro"/>
-  <xacro:macro name="pioneer3dx_body" params="meshes">
+  <xacro:macro name="pioneer3dx_body" params="name parent meshes">
     <!-- base_link -->
-    <link name="base_link"/>
+    <link name="${parent}"/>
     <!-- Chassis -->
-    <xacro:pioneer_chassis name="chassis" parent="base_link" xyz="0 0 0" rpy="0 0 0"  meshes="${meshes}"/>
+    <xacro:pioneer_chassis name="${name}" parent="base_link" xyz="0 0 0" rpy="0 0 0"  meshes="${meshes}"/>
     <!-- Front Sonar -->
-    <xacro:pioneer_sonar name="sonar" parent="chassis" xyz="0.109 0 0.209" rpy="0 0 0"  meshes="${meshes}"/>
+    <xacro:pioneer_sonar name="sonar" parent="${name}" xyz="0.109 0 0.209" rpy="0 0 0"  meshes="${meshes}"/>
     <!-- Akku0 -->
-    <xacro:battery_block name="battery0" parent="chassis" x="-0.14" y="0.00"  z="0.13" mass="2.5" />
+    <xacro:battery_block name="battery0" parent="${name}" x="-0.14" y="0.00"  z="0.13" mass="2.5" />
     <!-- Wheels -->
-    <xacro:pioneer_wheel side="right" parent="chassis"  xyz="0  0.15 0.09" rpy="0 0 0" radius="0.09" meshes="${meshes}"/>
-    <xacro:pioneer_wheel side="left"  parent="chassis"  xyz="0 -0.15 0.09" rpy="0 0 0" radius="0.09" meshes="${meshes}"/>
-    <xacro:pioneer_swivel parent="chassis"  xyz="-0.185 0 0.055" rpy="0 0 0" meshes="${meshes}"/>
+    <xacro:pioneer_wheel side="right" parent="${name}"  xyz="0  0.15 0.09" rpy="0 0 0" radius="0.09" meshes="${meshes}"/>
+    <xacro:pioneer_wheel side="left"  parent="${name}"  xyz="0 -0.15 0.09" rpy="0 0 0" radius="0.09" meshes="${meshes}"/>
+    <xacro:pioneer_swivel parent="${name}"  xyz="-0.185 0 0.055" rpy="0 0 0" meshes="${meshes}"/>
     <!-- Motor plugin -->
     <xacro:pioneer3dx_diff_drive />
