Commit message: debug of tricycle drive:  - broadcast of vel_current and vel_target  - controller bugs  - odometry bugs  - now v and w represent in all topics linear velocity and angle of actuated wheel

File: gazebo_plugins/test/tricycle_drive/xacro/tricycle/wheel_actuated.xacro (robot description, xacro)
@@ -27,4 +27,36 @@
   </gazebo>
   <!-- wheel joint -->
+  <joint name="${side}_wheel_joint" type="fixed">
+    <axis xyz="0 1 0"/>
+    <origin xyz="0 0 0" rpy="0 0 0"/>
+    <parent link="${side}_steering_joint"/>
+    <child link="${side}_wheel"/>
+  </joint>
+  <link name="${side}_wheel">
+    <inertial>
+      <mass value="0.5"/>
+      <origin xyz="0 0 0"/>
+      <inertia ixx="0.012411765597" ixy="0" ixz="0" iyy="0.015218160428" iyz="0" izz="0.011763977943"/>
+    </inertial>
+    <visual name="base_visual">
+      <origin xyz="0 0 0" rpy="0 0 0"/>
+      <geometry name="pioneer_geom">
+        <mesh filename="${meshes}/${side}_wheel.stl"/>
+      </geometry>
+      <material name="WheelBlack">
+        <color rgba="0.117 0.117 0.117 1"/>
+      </material>
+    </visual>
+    <collision>
+      <origin xyz="0 0 0" rpy="${-3.1415927/2} 0 0"/>
+      <geometry>
+        <!--<mesh filename="${meshes}/${side}_wheel.stl"/>-->
+        <cylinder radius="${radius}" length="0.01"/>
+      </geometry>
+    </collision>
+  </link>
+  <gazebo reference="${side}_wheel">
+    <material value="Gazebo/Black"/>
+  </gazebo>
   <xacro:wheel name="${name}"  parent="${name}_steering"  xyz="0 0 0" rpy="0 0 0" radius="${radius}" length="${length}" meshes="${meshes}"/>
   </xacro:macro>
