Commit message: diffdrive fixed and test environment added

File: gazebo_plugins/test/pioneer3dx/xacro/pioneer3dx/battery_block.xacro (robot description, xacro)
@@ -1,5 +1,5 @@
 <?xml version="1.0"?>
-<robot xmlns:xacro="http://ros.org/wiki/xacro">
-  <property name="M_PI" value="3.1415926535897931" />
+<robot xmlns:xacro="http://www.ros.org/wiki/xacro">
+  <xacro:property name="M_PI" value="3.1415926535897931" />
   <xacro:macro name="battery_block" params="name parent x y z mass">
   <joint name="${parent}_${name}_joint" type="fixed">

File: gazebo_plugins/test/pioneer3dx/xacro/pioneer3dx/inertia_tensors.xacro (robot description, xacro)
@@ -3,6 +3,6 @@
   see https://github.com/uos/uos_tools/blob/fuerte/uos_common_urdf/common.xacro and
   see http://answers.gazebosim.org/question/4372/the-inertia-matrix-explained/ -->
-<robot xmlns:xacro="http://ros.org/wiki/xacro">
-  <property name="M_PI" value="3.1415926535897931" />
+<robot xmlns:xacro="http://www.ros.org/wiki/xacro">
+  <xacro:property name="M_PI" value="3.1415926535897931" />
   <!-- see https://secure.wikimedia.org/wikipedia/en/wiki/List_of_moment_of_inertia_tensors -->
   <!-- #################### versions without origin #################### -->
@@ -38,5 +38,5 @@
     <inertial>
       <mass value="${mass}" />
-      <insert_block name="origin" />
+      <xacro:insert_block name="origin" />
       <inertia ixx="${0.4 * mass * radius * radius}" ixy="0.0" ixz="0.0"
         iyy="${0.4 * mass * radius * radius}" iyz="0.0"
@@ -47,5 +47,5 @@
     <inertial>
       <mass value="${mass}" />
-      <insert_block name="origin" />
+      <xacro:insert_block name="origin" />
       <inertia ixx="${0.0833333 * mass * (3 * radius * radius + length * length)}" ixy="0.0" ixz="0.0"
         iyy="${0.0833333 * mass * (3 * radius * radius + length * length)}" iyz="0.0"
@@ -56,5 +56,5 @@
     <inertial>
       <mass value="${mass}" />
-      <insert_block name="origin" />
+      <xacro:insert_block name="origin" />
       <inertia ixx="${0.0833333 * mass * (y*y + z*z)}" ixy="0.0" ixz="0.0"
         iyy="${0.0833333 * mass * (x*x + z*z)}" iyz="0.0"

File: gazebo_plugins/test/pioneer3dx/xacro/pioneer3dx/pioneer3dx_chassis.xacro (robot description, xacro)
@@ -1,5 +1,5 @@
 <?xml version="1.0"?>
-<robot xmlns:xacro="http://ros.org/wiki/xacro">
-  <property name="M_PI" value="3.1415926535897931" />
+<robot xmlns:xacro="http://www.ros.org/wiki/xacro">
+  <xacro:property name="M_PI" value="3.1415926535897931" />
   <xacro:macro name="pioneer_chassis" params="name parent xyz rpy meshes">
   <!-- Chassis -->
@@ -13,5 +13,5 @@
       <origin xyz="-0.045 0 0.148" rpy="0 0 0"/>
       <geometry name="pioneer_geom">
-        <mesh filename="${meshes}/chassis.stl"/>
+        <mesh filename="${meshes}/chassis.dae"/>
       </geometry>
       <material name="ChassisRed">
@@ -22,5 +22,5 @@
       <origin xyz="-0.045 0 0.148" rpy="0 0 0"/>
       <geometry>
-        <mesh filename="${meshes}/chassis.stl"/>
+        <mesh filename="${meshes}/chassis.dae"/>
       </geometry>
     </collision>
@@ -40,5 +40,5 @@
       <origin xyz="0 0 0" rpy="0 0 0"/>
       <geometry name="top_geom">
-        <mesh filename="${meshes}/top.stl"/>
+        <mesh filename="${meshes}/top.dae"/>
       </geometry>
       <material name="TopBlack">
@@ -49,5 +49,5 @@
     <origin xyz="0.0 0 0.0" rpy="0 0 0"/>
       <geometry>
-        <mesh filename="${meshes}/top.stl"/>
+        <mesh filename="${meshes}/top.dae"/>
       </geometry>
     </collision>

File: gazebo_plugins/test/pioneer3dx/xacro/pioneer3dx/pioneer3dx_sonar.xacro (robot description, xacro)
@@ -1,5 +1,5 @@
 <?xml version="1.0"?>
-<robot xmlns:xacro="http://ros.org/wiki/xacro">
-  <property name="M_PI" value="3.1415926535897931" />
+<robot xmlns:xacro="http://www.ros.org/wiki/xacro">
+  <xacro:property name="M_PI" value="3.1415926535897931" />
   <xacro:macro name="pioneer_sonar" params="name parent xyz rpy meshes">
   <!-- Front Sonar -->
@@ -18,5 +18,5 @@
       <origin xyz="0 0 0" rpy="0 0 0"/>
       <geometry name="pioneer_geom">
-        <mesh filename="${meshes}/back_sonar.stl"/>
+        <mesh filename="${meshes}/back_sonar.dae"/>
       </geometry>
       <material name="SonarYellow">

File: gazebo_plugins/test/pioneer3dx/xacro/pioneer3dx/pioneer3dx_swivel.xacro (robot description, xacro)
@@ -1,5 +1,5 @@
 <?xml version="1.0"?>
-<robot xmlns:xacro="http://ros.org/wiki/xacro">
-  <property name="M_PI" value="3.1415926535897931" />
+<robot xmlns:xacro="http://www.ros.org/wiki/xacro">
+  <xacro:property name="M_PI" value="3.1415926535897931" />
   <xacro:macro name="pioneer_swivel" params="parent xyz rpy meshes">
   <!-- Swivel -->

File: gazebo_plugins/test/pioneer3dx/xacro/pioneer3dx/pioneer3dx_wheel.xacro (robot description, xacro)
@@ -1,6 +1,6 @@
 <?xml version="1.0"?>
 <robot
-  xmlns:xacro="http://ros.org/wiki/xacro">
-  <property name="M_PI" value="3.1415926535897931" />
+  xmlns:xacro="http://www.ros.org/wiki/xacro">
+  <xacro:property name="M_PI" value="3.1415926535897931" />
   <xacro:macro name="pioneer_wheel" params="side parent xyz rpy radius meshes">
   <!-- Hubcap -->
@@ -20,5 +20,5 @@
       <origin xyz="0 0 0" rpy="0 0 0"/>
       <geometry name="pioneer_geom">
-        <mesh filename="${meshes}/${side}_hubcap.stl"/>
+        <mesh filename="${meshes}/hubcap.dae"/>
       </geometry>
       <material name="HubcapYellow">
@@ -52,5 +52,5 @@
       <origin xyz="0 0 0" rpy="0 0 0"/>
       <geometry name="pioneer_geom">
-        <mesh filename="${meshes}/${side}_wheel.stl"/>
+        <mesh filename="${meshes}/wheel.dae"/>
       </geometry>
       <material name="WheelBlack">

File: gazebo_plugins/test/tricycle_drive/xacro/tricycle/inertia_tensors.xacro (robot description, xacro)
@@ -3,5 +3,5 @@
   see https://github.com/uos/uos_tools/blob/fuerte/uos_common_urdf/common.xacro and
   see http://answers.gazebosim.org/question/4372/the-inertia-matrix-explained/ -->
-<robot xmlns:xacro="http://ros.org/wiki/xacro">
+<robot xmlns:xacro="http://www.ros.org/wiki/xacro">
   <property name="M_PI" value="3.1415926535897931" />
   <!-- see https://secure.wikimedia.org/wikipedia/en/wiki/List_of_moment_of_inertia_tensors -->

File: gazebo_plugins/test/tricycle_drive/xacro/tricycle/tricycle_chassis.xacro (robot description, xacro)
@@ -1,4 +1,4 @@
 <?xml version="1.0"?>
-<robot xmlns:xacro="http://ros.org/wiki/xacro">
+<robot xmlns:xacro="http://www.ros.org/wiki/xacro">
   <property name="M_PI" value="3.1415926535897931" />
   <property name="DX" value="2.500" />

File: gazebo_plugins/test/tricycle_drive/xacro/tricycle/wheel.xacro (robot description, xacro)
@@ -1,5 +1,5 @@
 <?xml version="1.0"?>
 <robot
-  xmlns:xacro="http://ros.org/wiki/xacro">
+  xmlns:xacro="http://www.ros.org/wiki/xacro">
   <property name="M_PI" value="3.1415926535897931" />
   <xacro:macro name="wheel" params="name parent xyz rpy radius length meshes">

File: gazebo_plugins/test/tricycle_drive/xacro/tricycle/wheel_actuated.xacro (robot description, xacro)
@@ -1,4 +1,4 @@
 <?xml version="1.0"?>
-<robot xmlns:xacro="http://ros.org/wiki/xacro">
+<robot xmlns:xacro="http://www.ros.org/wiki/xacro">
   <property name="M_PI" value="3.1415926535897931" />
   <xacro:macro name="wheel_actuated" params="name parent xyz rpy radius length meshes">

File: gazebo_plugins/test2/large_models/large_model.urdf.xacro (robot description, xacro)
@@ -12,5 +12,5 @@
        xmlns:renderable="http://playerstage.sourceforge.net/gazebo/xmlschema/#renderable"
        xmlns:controller="http://playerstage.sourceforge.net/gazebo/xmlschema/#controller"
-       xmlns:xacro="http://ros.org/wiki/xacro"
+       xmlns:xacro="http://www.ros.org/wiki/xacro"
        xmlns:physics="http://playerstage.sourceforge.net/gazebo/xmlschema/#physics">
   <link name="world"/>

File: gazebo_plugins/test2/large_models/smaller_large_model.urdf.xacro (robot description, xacro)
@@ -12,5 +12,5 @@
        xmlns:renderable="http://playerstage.sourceforge.net/gazebo/xmlschema/#renderable"
        xmlns:controller="http://playerstage.sourceforge.net/gazebo/xmlschema/#controller"
-       xmlns:xacro="http://ros.org/wiki/xacro"
+       xmlns:xacro="http://www.ros.org/wiki/xacro"
        xmlns:physics="http://playerstage.sourceforge.net/gazebo/xmlschema/#physics">
   <link name="world"/>
